File: luxmètre/luxmètre.kicad_sch (KiCad schematic)
At the start: 84 parts, among them J1 USB_A, J2 Conn_01x08, J3 Conn_01x01, J4 Conn_01x04, J5 Conn_01x01, J6 Conn_01x01, J7 Conn_01x03, J8 Conn_01x03, SW1 B3S-1000P, U1 ESP32-WROOM-32, U10 MAX1674EUA+T, U11 MCP73831-2-MC, U3 ADC-10-4+, U4 RF-LORA-868-SO, U5 PCA9537DP, U6 FT232HL, U7 ILB1206ER260V, U8 ILB1206ER260V, U9 ILB1206ER260V, Y1 12MHz

Commit message: routage computing unit bloc
Parts:
- removed JP2: Jumper_2_Open, Capacitor_SMD:CP_Elec_5x5.4, symbol Jumper:Jumper_2_Open
- added C23, C25: 10uF, Capacitor_SMD:C_0805_2012Metric_Pad1.18x1.45mm_HandSolder, symbol Device:C_Polarized_US
- added C27, C29: 100nF, Capacitor_SMD:C_0805_2012Metric_Pad1.18x1.45mm_HandSolder, symbol Device:C
- added C30: 10nF, Capacitor_SMD:C_0805_2012Metric_Pad1.18x1.45mm_HandSolder, symbol Device:C
- added D4, D5: BAT54C, Package_TO_SOT_SMD:SOT-23, symbol Diode:BAT54C
- added D8: LED, LED_SMD:LED_0805_2012Metric_Pad1.15x1.40mm_HandSolder, symbol Device:LED
- added J1, J10, J11, J13, J2: Conn_01x01, TestPoint:TestPoint_Loop_D2.50mm_Drill1.85mm, symbol Connector_Generic:Conn_01x01
- added J7: Conn_01x08, Connector_PinSocket_1.27mm:PinSocket_1x08_P1.27mm_Vertical, symbol Connector_Generic:Conn_01x08
- added J8: Conn_01x10, Connector_PinSocket_1.27mm:PinSocket_1x10_P1.27mm_Vertical, symbol Connector_Generic:Conn_01x10
- added J9: Conn_01x03, Connector_PinHeader_1.27mm:PinHeader_1x03_P1.27mm_Vertical, symbol Connector_Generic:Conn_01x03
- added JP3: Jumper_2_Open, Jumper:SolderJumper-2_P1.3mm_Bridged2Bar_RoundedPad1.0x1.5mm, symbol Jumper:Jumper_2_Open
- added R15: 0R1, Resistor_SMD:R_0805_2012Metric_Pad1.20x1.40mm_HandSolder, symbol Device:R
- added R17, R18: 330R, Resistor_SMD:R_0805_2012Metric_Pad1.20x1.40mm_HandSolder, symbol Device:R
- added SW2: SW_DIP_x01, Button_Switch_THT:SW_DIP_SPSTx01_Piano_10.8x4.1mm_W7.62mm_P2.54mm, symbol Switch:SW_DIP_x01
- added U11: AD8418, symbol Amplifier_Current:AD8418
- added U9: LM1117MP-3.3, Package_TO_SOT_SMD:SOT-223-3_TabPin2, symbol Regulator_Linear:LM1117MP-3.3
- U6: renamed from U2; footprint LED_SMD:LED_0805_2012Metric_Pad1.15x1.40mm_HandSolder -> OptoDevice:AMS_TSL25911FN
- renumbered C22 to C1, C14 to C10, C7 to C11, C16 to C12, C12 to C14, C11 to C15, C8 to C16, C1 to C17, C9 to C18, C10 to C19, C18 to C2, C3 to C20, C23 to C21, C24 to C22, C25 to C24, C2 to C26, C4 to C28, C5 to C3, C26 to C31, C17 to C4, C6 to C5, C20 to C6, C21 to C7, C15 to C8, C19 to C9, D2 to D1, D3 to D2, D1 to D3, D4 to D6, D5 to D7, J6 to J12, J5 to J14, J7 to J15, J8 to J16, J1 to J3, J3 to J4, J4 to J5, J2 to J6, JP4 to JP2, JP3 to JP4, R19 to R1, R14 to R10, R16 to R11, R21 to R12, R22 to R13, R25 to R14, R26 to R16, R1 to R19, R20 to R2, R5 to R20, R27 to R21, R8 to R22, R7 to R23, R6 to R24, R9 to R25, R10 to R26, R11 to R27, R12 to R28, R4 to R3, R3 to R4, R2 to R5, R15 to R6, R17 to R7, R13 to R8, R18 to R9, RF2 to RF1, U9 to U1, U4 to U10, U11 to U12, U3 to U13, U8 to U2, U7 to U3, U1 to U4, U6 to U5, U5 to U7, U10 to U8
Connections:
- net /RST is gone; now on net RST: C11.1, D3.1 (K), J4.1 (Pin_1), R8.2, SW1.3, SW1.4, U4.3 (EN), U7.6 (RESET/)
- net +3.3V: now also C27.1, C29.1, J11.1 (Pin_1), J7.2 (Pin_2), J7.4 (Pin_4), JP3.1 (A), R15.2, R17.1, U11.1 (IN-), U11.6 (VS)
- net 5V_BAT: now also J9.3 (Pin_3)
- net GND: now also C23.2, C25.2, C27.2, C29.2, C30.2, D8.1 (K), J10.1 (Pin_1), J7.6 (Pin_6), J7.7 (Pin_7), J8.4 (Pin_4), U11.2 (GND), U11.3 (REF2), U11.7 (REF1), U9.1 (GND)
- net MISO_L: now also J8.7 (Pin_7)
- net MOSI_L: now also J8.8 (Pin_8)
- net RXD: now also J1.1 (Pin_1), J8.6 (Pin_6)
- net SCK_L: now also J8.9 (Pin_9)
- net SCL: now also J8.1 (Pin_1)
- net SDA: now also J8.2 (Pin_2)
- net TXD: now also J2.1 (Pin_1), J8.5 (Pin_5)
- net VCC_USB: now also D4.1
- net /SS_L: now also J8.10 (Pin_10)
- net RST: now reaches U5.20 (ADBUS7)
- net RST: now also J7.3 (Pin_3), J8.3 (Pin_3)
- net at C26.1, C28.1, U10.3 (VCC): now also JP3.2 (B)
- new net: C30.1, J13.1 (Pin_1), R18.2
- new net: C25.1, R15.1, U11.8 (IN+), U9.2 (VO)
- new net: D4.3, D5.3, J9.1 (Pin_1)
- new net: J9.2 (Pin_2), SW2.1
- new net: R18.1, U11.5 (OUT)
- new net: D8.2 (A), R17.2
- new net +5V: C23.1, J7.5 (Pin_5), SW2.2, U9.3 (VI)
- new net VCC_EXT: D5.1, J7.8 (Pin_8)
- no-connect marks 42 -> 44
Other:
- note added: "Battery power"
- note added: "Computing Unit"
- note added: "Power select system"
- note added: "Sensors function"
- note added: "Wireless Transmission - LoRa"
- note removed: "Battery"
- moved on the sheet: BT1, C17, C20, C21, C22, C24, C26, C28, C31, D6, D7, J12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
