File: luxmètre/_autosave-luxmètre.kicad_sch (KiCad schematic)
At the start: 110 parts, among them J10 Conn_01x01, J11 Conn_01x01, J12 Conn_01x01, J13 Conn_01x01, J14 Conn_01x01, J15 Conn_01x03, J16 Conn_01x03, J3 USB_A, J4 Conn_01x01, J5 Conn_01x04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

Commit message: pcb
Connections:
- net GNDPWR: now also R1.1, R2.1
Other:
- note added: "Battery system"
- note removed: "Battery power"
Changed lines of the file:
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@@
 		)
 	)
-	(text "Battery power"
+	(text "Battery system"
 		(exclude_from_sim no)
 		(at 407.416 214.122 0)
@@
 	(text "USB Interface"
 		(exclude_from_sim no)
-		(at 121.666 142.748 0)
+		(at 83.566 149.352 0)
 		(effects
 			(font
@@
 	(symbol
 		(lib_id "power:GNDPWR")
-		(at 27.94 233.68 0)
+		(at 34.29 238.76 0)
 		(unit 1)
 		(exclude_from_sim no)
@@
 		(fields_autoplaced yes)
 		(property "Reference" "#PWR01"
-			(at 27.94 238.76 0)
+			(at 34.29 243.84 0)
 			(effects
 				(font
@@
 		)
 		(property "Value" "GNDPWR"
-			(at 27.813 237.49 0)
+			(at 34.163 242.57 0)
 			(effects
 				(font
@@
 		)
 		(property "Footprint" ""
-			(at 27.94 234.95 0)
+			(at 34.29 240.03 0)
 			(effects
 				(font
@@
 		)
 		(property "Datasheet" ""
-			(at 27.94 234.95 0)
+			(at 34.29 240.03 0)
 			(effects
 				(font
@@
 		)
 		(property "Description" "Power symbol creates a global label with name \"GNDPWR\" , global ground"
-			(at 27.94 233.68 0)
+			(at 34.29 238.76 0)
 			(effects
 				(font
