File: luxmètre/luxmètre.kicad_pcb (KiCad board)
At the start: 4 copper layers, 110.5 x 63 mm, 39 parts, among them J1 Conn_01x01, J2 Conn_01x01, J3 USB_A, J4 Conn_01x01, SW1 B3S-1000P, U10 RF-LORA-868-SO, U13 ADC-10-4+, U4 ESP32-WROOM-32, U7 PCA9537DP

Commit message: pcb
Parts:
- added BT1: Battery, Connector_Hirose:Hirose_DF13-02P-1.25DS_1x02_P1.25mm_Horizontal, F.Cu at (122.2, 60.0)
- added C1: 10uF, Capacitor_SMD:C_0805_2012Metric_Pad1.18x1.45mm_HandSolder, F.Cu at (59.0, 101.3)
- added C10: 100nF, Capacitor_SMD:C_0805_2012Metric_Pad1.18x1.45mm_HandSolder, F.Cu at (74.6, 95.1)
- added C12: 100nF, Capacitor_SMD:C_0805_2012Metric_Pad1.18x1.45mm_HandSolder, F.Cu at (77.5, 81.8)
- added C13: 100nF, Capacitor_SMD:C_0805_2012Metric_Pad1.18x1.45mm_HandSolder, F.Cu at (74.6, 97.2)
- added C14: 3.3uF, Capacitor_SMD:C_0805_2012Metric_Pad1.18x1.45mm_HandSolder, F.Cu at (93.3, 84.6)
- added C15: 100nF, Capacitor_SMD:C_0805_2012Metric_Pad1.18x1.45mm_HandSolder, F.Cu at (93.4, 87.3)
- added C16: 100nF, Capacitor_SMD:C_0805_2012Metric_Pad1.18x1.45mm_HandSolder, F.Cu at (98.0, 95.0)
- added C18: 100nF, Capacitor_SMD:C_0805_2012Metric_Pad1.18x1.45mm_HandSolder, F.Cu at (93.6, 92.0)
- added C19: 100nF, Capacitor_SMD:C_0805_2012Metric_Pad1.18x1.45mm_HandSolder, F.Cu at (93.6, 95.0)
- added C2: 10uF, Capacitor_SMD:C_0805_2012Metric_Pad1.18x1.45mm_HandSolder, F.Cu at (86.7, 84.5)
- added C21: 100nF, Capacitor_SMD:C_0805_2012Metric_Pad1.18x1.45mm_HandSolder, F.Cu at (142.6, 100.9)
- added C22: 100nF, Capacitor_SMD:C_0805_2012Metric_Pad1.18x1.45mm_HandSolder, F.Cu at (130.2, 78.9)
- added C23: 10uF, Capacitor_SMD:C_0805_2012Metric_Pad1.18x1.45mm_HandSolder, F.Cu at (110.8, 97.4)
- added C24: 47uF, Capacitor_SMD:CP_Elec_5x5.4, F.Cu at (132.7, 85.3)
- added C25: 10uF, Capacitor_SMD:C_0805_2012Metric_Pad1.18x1.45mm_HandSolder, F.Cu at (110.8, 95.0)
- added C27: 100nF, Capacitor_SMD:C_0805_2012Metric_Pad1.18x1.45mm_HandSolder, F.Cu at (106.4, 97.4)
- added C29: 100nF, Capacitor_SMD:C_0805_2012Metric_Pad1.18x1.45mm_HandSolder, F.Cu at (111.9, 84.9)
- added C30: 10nF, Capacitor_SMD:C_0805_2012Metric_Pad1.18x1.45mm_HandSolder, F.Cu at (125.4, 86.1)
- added C31: 47uF, Capacitor_SMD:CP_Elec_5x5.4, F.Cu at (132.9, 92.4)
- added C4: 10uF, Capacitor_SMD:C_0805_2012Metric_Pad1.18x1.45mm_HandSolder, F.Cu at (77.5, 84.3)
- added C6: 10nF, Capacitor_SMD:C_0805_2012Metric_Pad1.18x1.45mm_HandSolder, F.Cu at (75.1, 86.8)
- added C7: 10nF, Capacitor_SMD:C_0805_2012Metric_Pad1.18x1.45mm_HandSolder, F.Cu at (71.4, 88.1)
- added C8: 100nF, Capacitor_SMD:C_0805_2012Metric_Pad1.18x1.45mm_HandSolder, F.Cu at (86.7, 82.1)
- added C9: 10nF, Capacitor_SMD:C_0805_2012Metric_Pad1.18x1.45mm_HandSolder, F.Cu at (98.0, 92.1)
- added D2: PGB102ST23WR, easyeda2kicad:SOT-23_L3.0-W2.2-P0.95-LS2.2-TR, F.Cu at (71.0, 91.8)
- added D4: BAT54C, Package_TO_SOT_SMD:SOT-23, F.Cu at (125.9, 93.0)
- added D5: BAT54C, Package_TO_SOT_SMD:SOT-23, F.Cu at (125.8, 97.0)
- added D6: MBR0520LT, Diode_SMD:D_SOD-123F, F.Cu at (130.1, 76.5)
- added D7: LED, LED_SMD:LED_0805_2012Metric_Pad1.15x1.40mm_HandSolder, F.Cu at (132.7, 97.5)
- added D8: LED, LED_SMD:LED_0805_2012Metric_Pad1.15x1.40mm_HandSolder, F.Cu at (106.4, 95.0)
- added H1: MountingHole, MountingHole:MountingHole_2.2mm_M2_DIN965_Pad, F.Cu at (51.2, 103.9)
- added H2: MountingHole, MountingHole:MountingHole_2.2mm_M2_DIN965_Pad, F.Cu at (153.3, 44.3)
- added H3: MountingHole, MountingHole:MountingHole_2.2mm_M2_DIN965_Pad, F.Cu at (154.4, 103.7)
- added H4: MountingHole, MountingHole:MountingHole_2.2mm_M2_DIN965_Pad, F.Cu at (52.5, 43.9)
- added J10: Conn_01x01, TestPoint:TestPoint_Loop_D2.50mm_Drill1.85mm, F.Cu at (90.1, 102.4)
- added J11: Conn_01x01, TestPoint:TestPoint_Loop_D2.50mm_Drill1.85mm, F.Cu at (85.1, 102.5)
- added J12: Conn_01x01, TestPoint:TestPoint_Loop_D2.50mm_Drill1.85mm, F.Cu at (137.8, 96.7)
- added J13: Conn_01x01, TestPoint:TestPoint_Loop_D2.50mm_Drill1.85mm, F.Cu at (125.3, 82.3)
- added J14: Conn_01x01, TestPoint:TestPoint_Loop_D2.50mm_Drill1.85mm, F.Cu at (151.9, 67.5)
- added J15: Conn_01x03, Connector_Hirose:Hirose_DF13-03P-1.25DS_1x03_P1.25mm_Horizontal, F.Cu at (150.9, 49.7)
- added J16: Conn_01x03, Connector_Hirose:Hirose_DF13-03P-1.25DS_1x03_P1.25mm_Horizontal, F.Cu at (150.9, 56.3)
- added J5: Conn_01x04, Connector_PinSocket_1.27mm:PinSocket_1x08_P1.27mm_Vertical, F.Cu at (114.1, 50.0)
- added J6: Conn_01x08, Connector_PinSocket_1.27mm:PinSocket_1x08_P1.27mm_Vertical, F.Cu at (102.4, 50.0)
- added J7: Conn_01x08, Connector_PinSocket_1.27mm:PinSocket_1x08_P1.27mm_Vertical, F.Cu at (90.0, 49.8)
- added J8: Conn_01x10, Connector_PinSocket_1.27mm:PinSocket_1x10_P1.27mm_Vertical, F.Cu at (76.1, 49.8)
- added J9: Conn_01x03, Connector_PinHeader_1.27mm:PinHeader_1x03_P1.27mm_Vertical, F.Cu at (124.0, 101.9)
- added L1: 22uH, Inductor_SMD:L_6.3x6.3_H3, F.Cu at (139.9, 84.9)
- added R1: V5.5MLA0603NH, easyeda2kicad:R0603, F.Cu at (58.6, 99.5)
- added R11: 47k, Resistor_SMD:R_0805_2012Metric_Pad1.20x1.40mm_HandSolder, F.Cu at (93.5, 89.5)
- added R12: 113k, Resistor_SMD:R_0805_2012Metric_Pad1.20x1.40mm_HandSolder, F.Cu at (145.2, 78.8)
- added R13: 100k, Resistor_SMD:R_0805_2012Metric_Pad1.20x1.40mm_HandSolder, F.Cu at (145.2, 76.6)
- added R14: 100k, Resistor_SMD:R_0805_2012Metric_Pad1.20x1.40mm_HandSolder, F.Cu at (138.4, 74.8)
- added R15: 0R1, Resistor_SMD:R_0805_2012Metric_Pad1.20x1.40mm_HandSolder, F.Cu at (110.8, 92.6)
- added R16: 1.5k, Resistor_SMD:R_0805_2012Metric_Pad1.20x1.40mm_HandSolder, F.Cu at (132.6, 99.8)
- added R17: 330R, Resistor_SMD:R_0805_2012Metric_Pad1.20x1.40mm_HandSolder, F.Cu at (106.4, 92.6)
- added R18: 330R, Resistor_SMD:R_0805_2012Metric_Pad1.20x1.40mm_HandSolder, F.Cu at (125.4, 88.5)
- added R2: V5.5MLA0603NH, easyeda2kicad:R0603, F.Cu at (58.5, 103.1)
- added R21: 2k, Resistor_SMD:R_0805_2012Metric_Pad1.20x1.40mm_HandSolder, F.Cu at (132.6, 101.9)
- added R7: 10k, Resistor_SMD:R_0805_2012Metric_Pad1.20x1.40mm_HandSolder, F.Cu at (98.0, 89.4)
- added R9: 10k, Resistor_SMD:R_0805_2012Metric_Pad1.20x1.40mm_HandSolder, F.Cu at (74.7, 91.0)
- added SW2: SW_DIP_x01, Button_Switch_THT:SW_DIP_SPSTx01_Piano_10.8x4.1mm_W7.62mm_P2.54mm, F.Cu at (65.2, 102.5)
- added U1: ILB1206ER260V, easyeda2kicad:L1206, F.Cu at (55.7, 101.2)
- added U11: AD8418, Package_SO:SOIC-8-1EP_3.9x4.9mm_P1.27mm_EP2.29x3mm_ThermalVias, F.Cu at (118.2, 86.7)
- added U12: MCP73831-2-MC, Package_TO_SOT_SMD:SOT-23-5_HandSoldering, F.Cu at (137.7, 100.9)
- added U2: ILB1206ER260V, easyeda2kicad:L1206, F.Cu at (83.5, 82.9)
- added U3: ILB1206ER260V, easyeda2kicad:L1206, F.Cu at (80.9, 82.9)
- added U5: FT232HL, Package_QFP:LQFP-48_7x7mm_P0.5mm, F.Cu at (85.1, 90.9)
- added U8: MAX1674EUA+T, Converter_DCDC:Converter_DCDC_Cyntec_MUN12AD01-SH, F.Cu at (138.2, 78.0)
- added U9: LM1117MP-3.3, Package_TO_SOT_SMD:SOT-223-3_TabPin2, F.Cu at (118.2, 94.8)
- added Y1: 12MHz, Crystal:Crystal_SMD_2012-2Pin_2.0x1.2mm_HandSoldering, F.Cu at (75.0, 89.0)
- J3: footprint Connector_USB:USB_A_Molex_67643_Horizontal -> Connector_USB:USB_Micro-B_Molex_47346-0001
- JP1, JP2, JP3: footprint Jumper:SolderJumper-2_P1.3mm_Bridged2Bar_RoundedPad1.0x1.5mm -> Connector_PinHeader_1.27mm:PinHeader_1x02_P1.27mm_Vertical
- RF1: footprint Connector_Coaxial:SMA_Amphenol_901-144_Vertical -> easyeda2kicad:SMA-TH_HJ-2LC15SF048
- moved R27 110.4 mm to (90.5, 58.8), turned to 180 degrees
- moved R28 110.3 mm to (86.2, 58.8)
- moved R26 109.0 mm to (86.2, 61.3)
- moved R24 105.4 mm to (80.7, 69.1), turned to -90 degrees
- moved R25 104.3 mm to (86.2, 63.7)
- moved R23 103.8 mm to (90.5, 61.3)
- moved R22 99.0 mm to (90.5, 63.7), turned to 180 degrees
- moved U13 92.1 mm to (88.2, 70.4), turned to 90 degrees
- moved JP4 84.1 mm to (152.3, 63.6)
- moved U10 81.8 mm to (108.5, 65.2), turned to 90 degrees
- moved RF1 69.8 mm to (152.3, 74.7), turned to 90 degrees
- moved R20 66.8 mm to (109.7, 79.4), turned to 90 degrees
- moved R19 65.1 mm to (107.2, 79.4), turned to 90 degrees
- moved C26 63.7 mm to (104.6, 79.3), turned to -90 degrees
- moved C28 62.3 mm to (102.2, 79.3), turned to -90 degrees
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Routing:
- net /RST: track 0.00 -> 143.8 mm, vias 0 -> 6
- net V_BAT: track 0.00 -> 140.2 mm, vias 0 -> 2
- net +5V: track 0.00 -> 118.5 mm, vias 0 -> 2
- net GND: track 0.00 -> 110.7 mm, vias 0 -> 76
- net /TXD: track 0.00 -> 102.2 mm, vias 0 -> 8
- net Net-(JP4-SIG): track 0.00 -> 101.9 mm, vias 0 -> 4
- net /RXD: track 0.00 -> 98.6 mm, vias 0 -> 6
- net VCC_USB: track 0.00 -> 97.6 mm, vias 0 -> 6
- net Net-(U13-OUTPUT): track 0.00 -> 81.7 mm
- net /BOOT: track 0.00 -> 81.3 mm, vias 0 -> 8
- net /TX_SW: track 0.00 -> 79.3 mm, vias 0 -> 4
- net /RX_SW: track 0.00 -> 71.2 mm, vias 0 -> 4
- net /SCK_L: track 0.00 -> 67.9 mm, vias 0 -> 2
- net VCC_EXT: track 0.00 -> 67.9 mm, vias 0 -> 2
- net Net-(J9-Pin_2): track 0.00 -> 66.2 mm
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- added copper zone on In2.Cu, net +3.3V
- added copper zone on In1.Cu, net GND
- removed copper zone on B.Cu, net GND
Other:
- board size 110.5 x 63 mm -> 108.9 x 64.9 mm
- board text added: "+3.3V"
- board text added: "+5V"
- board text added: "/RST"
- board text added: "/SS_L"
- board text added: "Battery"
- board text added: "DIO0"
- board text added: "DIO1"
- board text added: "DIO2"
- board text added: "DIO3"
- board text added: "DIO4"
- board text added: "DIO5"
- board text added: "GND"
- board text added: "KOROTA"
- board text added: "MISO_L"
- board text added: "MOSI_L"
- board text added: "RF-LORA-868-SO"
- board text added: "RST"
- board text added: "RST_L"
- board text added: "RXD"
- board text added: "RX_SW"
- board text added: "SCK_L"
- board text added: "SCL"
- board text added: "SDA"
- board text added: "TXD"
- board text added: "TX_SW"
- board text added: "VCC_EXT"

Commit message: pcb
Other:
- board size 108.9 x 64.9 mm -> 108.2 x 64.2 mm
Changed lines of the file:
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@@
 			(outputformat 1)
 			(mirror no)
-			(drillshape 1)
+			(drillshape 0)
 			(scaleselection 1)
 			(outputdirectory "")
@@
 	)
 	(gr_rect
-		(start 48.63 41.75)
-		(end 157.51 106.66)
+		(start 49.3 41.75)
+		(end 157.51 106)
 		(stroke
 			(width 0.05)
@@
 		(polygon
 			(pts
-				(xy 49.82 45.69) (xy 158.42 45.5) (xy 158.21 104.88) (xy 49.58 105.29)
+				(xy 48.42 41.69) (xy 157.02 41.5) (xy 158.51 105.98) (xy 49.88 106.39)
 			)
 		)
@@
 		(polygon
 			(pts
-				(xy 49.6 46.42) (xy 158.63 45.55) (xy 157.98 104.37) (xy 49.57 105.25)
+				(xy 49 42.12) (xy 158.03 41.25) (xy 157.78 105.67) (xy 49.37 106.55)
 			)
 		)
